Commit message: bfok_0

File: resources/robots/zsl1/urdf/zsl1.urdf (robot description, URDF)
Before this commit: robot zsl1, 18 links, 17 joints
Links:
- removed link payload
- link FL_foot: geometry collision sphere radius=0.0295; visual mesh filename=../meshes/FL_FOOT_LINK.STL
- link FR_foot: geometry collision sphere radius=0.0295; visual mesh filename=../meshes/FR_FOOT_LINK.STL
- link RL_foot: geometry collision sphere radius=0.0295; visual mesh filename=../meshes/RL_FOOT_LINK.STL
- link RR_foot: geometry collision sphere radius=0.0295; visual mesh filename=../meshes/RR_FOOT_LINK.STL
Joints:
- removed joint pl_joint
